File: dasa-3/dasa-3.sch (KiCad schematic (older format))
At the start: 12 parts, among them J1 DB9_Male, J2 AVR-ISP-10, J3 AVR-ISP-6, Q1 BC546

Commit message: fix: update project
Connections:
- net TxD: now reaches J1.3, R1.2
- net DTR: now reaches J1.4, R3.2
- net RTS: now reaches J1.7, R2.2
- net CTS: now reaches J1.8, J2.9 (MISO), J3.1 (MISO)
Other:
- note added: "programmed avr powered form own circuit"
Changed lines of the file:
@@
 Wire Wire Line
 	4200 4370 4680 4370
+Text Label 3820 2830 0    50   ~ 0
+DTR
+Text Label 3820 2930 0    50   ~ 0
+CTS
+Text Label 3820 3030 0    50   ~ 0
+TxD
+Text Label 3820 3130 0    50   ~ 0
+RTS
+Text Label 3810 2630 0    50   ~ 0
+GND
+Text Notes 6490 4920 0    50   ~ 0
+programmed avr powered form own circuit
 $EndSCHEMATC
