File: dasa-3/dasa-3.kicad_pcb (KiCad board)
At the start: 2 copper layers, 31.5 x 63.5 mm, 12 parts, among them J1 DB9_Male, J2 AVR-ISP-10, J3 AVR-ISP-6, Q1 BC546

Commit message: update: update project files
Signed-off-by: Paweł Sobótka <48721262935pl@gmail.com>
Routing:
- removed copper zone on F.Cu, net GND
Changed lines of the file:
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@@
-(kicad_pcb (version 20171130) (host pcbnew 5.1.2-1.fc30)
+(kicad_pcb (version 20171130) (host pcbnew 5.1.4-3.fc30)
   (general
     (thickness 1.6)
-    (drawings 7)
+    (drawings 8)
     (tracks 97)
     (zones 0)
@@
   (page A4)
   (title_block
-    (title "avr dasa-3 programmer PCB")
-    (date 2019-07-21)
-    (rev 0.5)
+    (title "AVR dasa-3 programmer PCB layout")
+    (date 2019-09-20)
+    (rev 1.0)
     (company "mgr inż. Paweł Sobótka")
+    (comment 1 "GNU GPLv3")
+    (comment 2 "Device AVR Serial Adapter")
   )
   (layers
@@
       (drillshape 0)
       (scaleselection 1)
-      (outputdirectory "grbv/"))
+      (outputdirectory "gerbv/"))
   )
   (net 0 "")
@@
     )
   )
+  (target plus (at 118.9609 87.85352) (size 5) (width 0.05) (layer Edge.Cuts))
   (gr_text "avr \"dasa-3\" programmer" (at 144.018 79.248 90) (layer Dwgs.User)
     (effects (font (size 1 1) (thickness 0.15)))
@@
   (segment (start 120.396 108.966) (end 134.366 108.966) (width 0.5) (layer B.Cu) (net 16))
   (segment (start 134.366 108.966) (end 136.906 106.426) (width 0.5) (layer B.Cu) (net 16))
-  (zone (net 1) (net_name GND) (layer F.Cu) (hatch edge 0.508)
-    (connect_pads (clearance 0.508))
-    (min_thickness 0.254)
-    (fill yes (arc_segments 32) (thermal_gap 0.508) (thermal_bridge_width 0.508) (smoothing chamfer) (radius 3))
-    (polygon
-      (pts
-        (xy 116.586 48.006) (xy 116.586 111.506) (xy 148.082 111.506) (xy 148.082 48.006)
-      )
-    )
-  )
 )

Commit message: update: prepare Gerber files for productions
Changed lines of the file:
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@@
   (general
     (thickness 1.6)
-    (drawings 8)
+    (drawings 10)
     (tracks 97)
     (zones 0)
@@
     (visible_elements FFFFFF7F)
     (pcbplotparams
-      (layerselection 0x211fc_ffffffff)
+      (layerselection 0x291f0_ffffffff)
       (usegerberextensions false)
       (usegerberattributes false)
@@
       (viasonmask false)
       (mode 1)
-      (useauxorigin false)
+      (useauxorigin true)
       (hpglpennumber 1)
       (hpglpenspeed 20)
@@
       (plotinvisibletext false)
       (padsonsilk false)
-      (subtractmaskfromsilk false)
+      (subtractmaskfromsilk true)
       (outputformat 1)
       (mirror false)
@@
     )
   )
-  (target plus (at 118.9609 87.85352) (size 5) (width 0.05) (layer Edge.Cuts))
-  (gr_text "avr \"dasa-3\" programmer" (at 144.018 79.248 90) (layer Dwgs.User)
+  (dimension 63.506 (width 0.15) (layer Cmts.User)
+    (gr_text "63,506 mm" (at 153.7 79.753 90) (layer Cmts.User)
+      (effects (font (size 1 1) (thickness 0.15)))
+    )
+    (feature1 (pts (xy 148.082 48) (xy 152.986421 48)))
+    (feature2 (pts (xy 148.082 111.506) (xy 152.986421 111.506)))
+    (crossbar (pts (xy 152.4 111.506) (xy 152.4 48)))
+    (arrow1a (pts (xy 152.4 48) (xy 152.986421 49.126504)))
+    (arrow1b (pts (xy 152.4 48) (xy 151.813579 49.126504)))
+    (arrow2a (pts (xy 152.4 111.506) (xy 152.986421 110.379496)))
+    (arrow2b (pts (xy 152.4 111.506) (xy 151.813579 110.379496)))
+  )
+  (dimension 31.496 (width 0.15) (layer Cmts.User)
+    (gr_text "31,496 mm" (at 132.334 115.6) (layer Cmts.User)
+      (effects (font (size 1 1) (thickness 0.15)))
+    )
+    (feature1 (pts (xy 148.082 111.506) (xy 148.082 114.886421)))
+    (feature2 (pts (xy 116.586 111.506) (xy 116.586 114.886421)))
+    (crossbar (pts (xy 116.586 114.3) (xy 148.082 114.3)))
+    (arrow1a (pts (xy 148.082 114.3) (xy 146.955496 114.886421)))
+    (arrow1b (pts (xy 148.082 114.3) (xy 146.955496 113.713579)))
+    (arrow2a (pts (xy 116.586 114.3) (xy 117.712504 114.886421)))
+    (arrow2b (pts (xy 116.586 114.3) (xy 117.712504 113.713579)))
+  )
+  (target plus (at 146.05 109.22) (size 5) (width 0.05) (layer Edge.Cuts))
+  (gr_text "avr \"dasa-3\" programmer" (at 144.018 79.248 90) (layer F.SilkS)
     (effects (font (size 1 1) (thickness 0.15)))
   )
-  (target plus (at 144.526 52.07) (size 5) (width 0.05) (layer Edge.Cuts))
+  (target plus (at 119.38 50.8) (size 5) (width 0.05) (layer Edge.Cuts))
   (gr_line (start 116.586 48) (end 116.586 53.34) (layer Edge.Cuts) (width 0.05))
   (gr_line (start 116.586 111.506) (end 116.586 53.34) (layer Edge.Cuts) (width 0.05))
