File: bsd_programmer/bsd_programmer.kicad_pcb (KiCad board)
At the start: 2 copper layers, 50.3 x 54.6 mm, 12 parts, among them J1 DB25_Male, J2 AVR-ISP-10, M1 MountingHole_2.5mm, M2 MountingHole_2.5mm

Commit message: update: prepare Gerber files for productions
Parts:
- removed M1, M2: MountingHole_2.5mm, MountingHole:MountingHole_2.5mm
- added H1: M2.5, MountingHole:MountingHole_2.5mm, F.Cu at (177.8, 111.8)
- added H1: M2.5, MountingHole:MountingHole_2.5mm, F.Cu at (177.8, 68.6)
Connections:
- net MISO renamed ACK
- net MOSI renamed D7
- net RST renamed D5
- net SCK renamed D6
Changed lines of the file:
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@@
   (general
     (thickness 1.6)
-    (drawings 4)
+    (drawings 6)
     (tracks 57)
     (zones 0)
@@
     (pad_to_mask_clearance 0.051)
     (solder_mask_min_width 0.25)
-    (aux_axis_origin 0 0)
+    (aux_axis_origin 133.08 117.602)
     (visible_elements FFFFFF7F)
     (pcbplotparams
-      (layerselection 0x010a8_ffffffff)
+      (layerselection 0x292a8_ffffffff)
       (usegerberextensions false)
-      (usegerberattributes false)
-      (usegerberadvancedattributes false)
-      (creategerberjobfile false)
+      (usegerberattributes true)
+      (usegerberadvancedattributes true)
+      (creategerberjobfile true)
       (excludeedgelayer true)
-      (linewidth 0.100000)
+      (linewidth 0.150000)
       (plotframeref false)
       (viasonmask false)
       (mode 1)
-      (useauxorigin false)
+      (useauxorigin true)
       (hpglpennumber 1)
       (hpglpenspeed 20)
@@
       (plotinvisibletext false)
       (padsonsilk false)
-      (subtractmaskfromsilk false)
+      (subtractmaskfromsilk true)
       (outputformat 1)
       (mirror false)
@@
   (net 19 D2)
   (net 20 D3)
-  (net 21 RST)
-  (net 22 SCK)
-  (net 23 MOSI)
-  (net 24 MISO)
+  (net 21 D5)
+  (net 22 D6)
+  (net 23 D7)
+  (net 24 ACK)
   (net_class Default "To jest domyślna klasa połączeń."
     (clearance 0.2)
@@
     (uvia_dia 0.3)
     (uvia_drill 0.1)
+    (add_net ACK)
+    (add_net D5)
+    (add_net D6)
+    (add_net D7)
   )
   (net_class standard ""
@@
     (add_net D2)
     (add_net D3)
-    (add_net MISO)
-    (add_net MOSI)
     (add_net "Net-(J1-Pad1)")
     (add_net "Net-(J1-Pad11)")
@@
     (add_net "Net-(J2-Pad7)")
     (add_net "Net-(J2-Pad9)")
-    (add_net RST)
-    (add_net SCK)
   )
   (module MountingHole:MountingHole_2.5mm (layer F.Cu)
-    (at 177.292 112.014)
+    (at 177.8 111.76)
     (descr "Mounting Hole 2.5mm, no annular")
     (tags "mounting hole 2.5mm no annular")
     (attr virtual)
-    (fp_text reference M2 (at 0 -3.5) (layer F.SilkS)
-      (effects (font (size 1 1) (thickness 0.15)))
-    )
-    (fp_text value MountingHole_2.5mm (at -2.286 3.5) (layer F.Fab)
-      (effects (font (size 1 1) (thickness 0.15)))
-    )
+    (fp_text reference H1 (at 0 -3.5) (layer F.SilkS)
+      (effects (font (size 1 1) (thickness 0.15)))
+    )
+    (fp_text value M2.5 (at 0 3.5) (layer F.Fab)
+      (effects (font (size 1 1) (thickness 0.15)))
+    )
+    (fp_text user %R (at 0.3 0) (layer F.Fab)
+      (effects (font (size 1 1) (thickness 0.15)))
+    )
+    (fp_circle (center 0 0) (end 2.5 0) (layer Cmts.User) (width 0.15))
     (fp_circle (center 0 0) (end 2.75 0) (layer F.CrtYd) (width 0.05))
-    (fp_circle (center 0 0) (end 2.5 0) (layer Cmts.User) (width 0.15))
-    (fp_text user %R (at 0.3 0) (layer F.Fab)
-      (effects (font (size 1 1) (thickness 0.15)))
-    )
     (pad 1 np_thru_hole circle (at 0 0) (size 2.5 2.5) (drill 2.5) (layers *.Cu *.Mask))
   )
   (module MountingHole:MountingHole_2.5mm (layer F.Cu)
-    (at 177.038 68.834)
+    (at 177.8 68.58)
     (descr "Mounting Hole 2.5mm, no annular")
     (tags "mounting hole 2.5mm no annular")
     (attr virtual)
-    (fp_text reference M1 (at 0 -3.5) (layer F.SilkS)
-      (effects (font (size 1 1) (thickness 0.15)))
-    )
-    (fp_text value MountingHole_2.5mm (at -3.048 3.556) (layer F.Fab)
+    (fp_text reference H1 (at 0 -3.5) (layer F.SilkS)
+      (effects (font (size 1 1) (thickness 0.15)))
+    )
+    (fp_text value M2.5 (at 0 3.5) (layer F.Fab)
       (effects (font (size 1 1) (thickness 0.15)))
     )
@@
       (net 2 "Net-(J1-Pad6)"))
     (pad 7 thru_hole circle (at 16.62 0 270) (size 1.6 1.6) (drill 1) (layers *.Cu *.Mask)
-      (net 21 RST))
+      (net 21 D5))
     (pad 8 thru_hole circle (at 19.39 0 270) (size 1.6 1.6) (drill 1) (layers *.Cu *.Mask)
-      (net 22 SCK))
+      (net 22 D6))
     (pad 9 thru_hole circle (at 22.16 0 270) (size 1.6 1.6) (drill 1) (layers *.Cu *.Mask)
-      (net 23 MOSI))
+      (net 23 D7))
     (pad 10 thru_hole circle (at 24.93 0 270) (size 1.6 1.6) (drill 1) (layers *.Cu *.Mask)
-      (net 24 MISO))
+      (net 24 ACK))
     (pad 11 thru_hole circle (at 27.7 0 270) (size 1.6 1.6) (drill 1) (layers *.Cu *.Mask)
       (net 3 "Net-(J1-Pad11)"))
@@
       (net 16 "Net-(J2-Pad9)"))
     (pad 2 thru_hole oval (at 10.16 0 180) (size 1.6 1.6) (drill 0.8) (layers *.Cu *.Mask)
-      (net 24 MISO))
+      (net 24 ACK))
     (model ${KISYS3DMOD}/Resistor_THT.3dshapes/R_Axial_DIN0207_L6.3mm_D2.5mm_P10.16mm_Horizontal.wrl
       (at (xyz 0 0 0))
@@
     (fp_line (start 1.93 -1.25) (end 1.93 1.25) (layer F.Fab) (width 0.1))
     (pad 2 thru_hole oval (at 10.16 0 180) (size 1.6 1.6) (drill 0.8) (layers *.Cu *.Mask)
-      (net 23 MOSI))
+      (net 23 D7))
     (pad 1 thru_hole circle (at 0 0 180) (size 1.6 1.6) (drill 0.8) (layers *.Cu *.Mask)
       (net 11 "Net-(J2-Pad1)"))
@@
       (net 15 "Net-(J2-Pad7)"))
     (pad 2 thru_hole oval (at 10.16 0 180) (size 1.6 1.6) (drill 0.8) (layers *.Cu *.Mask)
-      (net 22 SCK))
+      (net 22 D6))
     (model ${KISYS3DMOD}/Resistor_THT.3dshapes/R_Axial_DIN0207_L6.3mm_D2.5mm_P10.16mm_Horizontal.wrl
       (at (xyz 0 0 0))
@@
     (fp_line (start 1.93 -1.25) (end 1.93 1.25) (layer F.Fab) (width 0.1))
     (pad 2 thru_hole oval (at 10.16 0 180) (size 1.6 1.6) (drill 0.8) (layers *.Cu *.Mask)
-      (net 21 RST))
+      (net 21 D5))
     (pad 1 thru_hole circle (at 0 0 180) (size 1.6 1.6) (drill 0.8) (layers *.Cu *.Mask)
       (net 14 "Net-(J2-Pad5)"))
@@
     )
   )
+  (dimension 54.61 (width 0.15) (layer Cmts.User)
+    (gr_text "54,610 mm" (at 191.8 90.297 90) (layer Cmts.User)
+      (effects (font (size 1 1) (thickness 0.15)))
+    )
+    (feature1 (pts (xy 183.388 62.992) (xy 191.086421 62.992)))
+    (feature2 (pts (xy 183.388 117.602) (xy 191.086421 117.602)))
+    (crossbar (pts (xy 190.5 117.602) (xy 190.5 62.992)))
+    (arrow1a (pts (xy 190.5 62.992) (xy 191.086421 64.118504)))
+    (arrow1b (pts (xy 190.5 62.992) (xy 189.913579 64.118504)))
+    (arrow2a (pts (xy 190.5 117.602) (xy 191.086421 116.475496)))
+    (arrow2b (pts (xy 190.5 117.602) (xy 189.913579 116.475496)))
+  )
+  (dimension 50.308 (width 0.15) (layer Cmts.User)
+    (gr_text "50,308 mm" (at 158.234 123.22) (layer Cmts.User)
+      (effects (font (size 1 1) (thickness 0.15)))
+    )
+    (feature1 (pts (xy 183.388 117.602) (xy 183.388 122.506421)))
+    (feature2 (pts (xy 133.08 117.602) (xy 133.08 122.506421)))
+    (crossbar (pts (xy 133.08 121.92) (xy 183.388 121.92)))
+    (arrow1a (pts (xy 183.388 121.92) (xy 182.261496 122.506421)))
+    (arrow1b (pts (xy 183.388 121.92) (xy 182.261496 121.333579)))
+    (arrow2a (pts (xy 133.08 121.92) (xy 134.206504 122.506421)))
+    (arrow2b (pts (xy 133.08 121.92) (xy 134.206504 121.333579)))
+  )
   (gr_line (start 133.08 117.602) (end 133.08 62.992) (layer Edge.Cuts) (width 0.05))
