File: bsd_programmer/bsd_programmer.sch (KiCad schematic (older format))
At the start: 10 parts, among them J1 DB25_Male, J2 AVR-ISP-10

Commit message: update: prepare Gerber files for productions
Parts:
- added H1: M2.5, MountingHole:MountingHole_2.5mm, symbol Mechanical:MountingHole
Changed lines of the file:
@@
 Text Notes 7120 2690 0    197  ~ 0
 Centronics pinouts
+$Comp
+L Mechanical:MountingHole H1
+U 1 1 5DA31830
+P 8050 4350
+F 0 "H1" H 8150 4396 50  0000 L CNN
+F 1 "M2.5" H 8150 4305 50  0000 L CNN
+F 2 "MountingHole:MountingHole_2.5mm" H 8050 4350 50  0001 C CNN
+F 3 "~" H 8050 4350 50  0001 C CNN
+	1    8050 4350
+	1    0    0    -1
+$EndComp
 $EndSCHEMATC
