File: dasa/dasa.kicad_pcb (KiCad board)
At the start: 2 copper layers, 46 x 81 mm, 16 parts, among them J1 DB9_Male, J2 AVR-ISP-10, J3 +5V

Commit message: update: update folder with new contents
Parts:
- J3: footprint Connector_BarrelJack:BarrelJack_Horizontal -> Connector_BarrelJack:BarrelJack_CUI_PJ-063AH_Horizontal
- moved J3 6.97 mm to (121.3, 108.2), turned to 270 degrees
- moved D6 3.04 mm to (115.8, 74.5)
- moved D1 3.02 mm to (115.8, 60.1)
- moved D5 3.00 mm to (132.6, 74.5)
- moved R4 3.00 mm to (151.6, 74.5)
- moved R1 2.92 mm to (115.7, 66.5)
- moved C1 2.64 mm to (145.2, 97.8)
- moved R2 2.44 mm to (115.7, 53.8)
- moved D4 2.34 mm to (115.8, 81.7)
- moved R3 2.13 mm to (115.7, 47.5)
- moved D3 2.08 mm to (132.6, 81.7)
- moved D7 0.15 mm to (132.6, 89.0)
- moved D8 0.15 mm to (115.8, 89.0)
Routing:
- net Net-(D7-Pad1): track 47.3 -> 36.0 mm
- net Net-(D8-Pad2): track 100.6 -> 106.3 mm
- net /RTS: track 32.1 -> 26.7 mm, vias 0 -> 1
- net Net-(D3-Pad1): track 91.5 -> 86.5 mm
- net /DSR: track 90.1 -> 94.9 mm, vias 0 -> 1
- net /DTR: track 16.0 -> 18.1 mm
- net /TxD: track 15.0 -> 16.7 mm
- net Net-(C1-Pad2): track 69.8 -> 71.0 mm
- net Net-(C1-Pad1): track 53.4 -> 52.9 mm

Commit message: update: prepare Gerber files for productions
Other:
- board text added: "avr "dasa" by SQ7EQE GNU GPLv3, 2019"
- board text removed: "avr "dasa""
Changed lines of the file:
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@@
   (general
     (thickness 1.6)
-    (drawings 6)
+    (drawings 9)
     (tracks 98)
     (zones 0)
@@
     (visible_elements FFFFFF7F)
     (pcbplotparams
-      (layerselection 0x213fc_ffffffff)
+      (layerselection 0x293f0_ffffffff)
       (usegerberextensions false)
-      (usegerberattributes false)
-      (usegerberadvancedattributes false)
+      (usegerberattributes true)
+      (usegerberadvancedattributes true)
       (creategerberjobfile true)
       (excludeedgelayer true)
-      (linewidth 0.100000)
+      (linewidth 0.150000)
       (plotframeref false)
       (viasonmask false)
       (mode 1)
-      (useauxorigin false)
+      (useauxorigin true)
       (hpglpennumber 1)
       (hpglpenspeed 20)
@@
       (plotinvisibletext false)
       (padsonsilk false)
-      (subtractmaskfromsilk false)
+      (subtractmaskfromsilk true)
       (outputformat 1)
       (mirror false)
@@
     )
   )
-  (target plus (at 137.16 43.18) (size 5) (width 0.05) (layer Edge.Cuts))
-  (gr_text "avr \"dasa\"" (at 117.094 41.402) (layer Dwgs.User)
+  (target plus (at 152.4 116.84) (size 5) (width 0.05) (layer Edge.Cuts))
+  (dimension 81.026 (width 0.15) (layer Cmts.User)
+    (gr_text "81,026 mm" (at 102.84 78.613 90) (layer Cmts.User)
+      (effects (font (size 1 1) (thickness 0.15)))
+    )
+    (feature1 (pts (xy 108.966 38.1) (xy 103.553579 38.1)))
+    (feature2 (pts (xy 108.966 119.126) (xy 103.553579 119.126)))
+    (crossbar (pts (xy 104.14 119.126) (xy 104.14 38.1)))
+    (arrow1a (pts (xy 104.14 38.1) (xy 104.726421 39.226504)))
+    (arrow1b (pts (xy 104.14 38.1) (xy 103.553579 39.226504)))
+    (arrow2a (pts (xy 104.14 119.126) (xy 104.726421 117.999496)))
+    (arrow2b (pts (xy 104.14 119.126) (xy 103.553579 117.999496)))
+  )
+  (dimension 45.974 (width 0.15) (layer Cmts.User)
+    (gr_text "45,974 mm" (at 131.953 123.22) (layer Cmts.User)
+      (effects (font (size 1 1) (thickness 0.15)))
+    )
+    (feature1 (pts (xy 154.94 119.126) (xy 154.94 122.506421)))
+    (feature2 (pts (xy 108.966 119.126) (xy 108.966 122.506421)))
+    (crossbar (pts (xy 108.966 121.92) (xy 154.94 121.92)))
+    (arrow1a (pts (xy 154.94 121.92) (xy 153.813496 122.506421)))
+    (arrow1b (pts (xy 154.94 121.92) (xy 153.813496 121.333579)))
+    (arrow2a (pts (xy 108.966 121.92) (xy 110.092504 122.506421)))
+    (arrow2b (pts (xy 108.966 121.92) (xy 110.092504 121.333579)))
+  )
+  (target plus (at 111.76 40.64) (size 5) (width 0.05) (layer Edge.Cuts))
+  (gr_text "avr \"dasa\" by SQ7EQE\nGNU GPLv3, 2019" (at 124.46 41.402) (layer F.SilkS)
     (effects (font (size 1 1) (thickness 0.15)))
   )
