File: usbasp/usbasp.sch (KiCad schematic (older format))
At the start: 26 parts, among them J1 USB_B, J2 TxD RxD, J3 AVR-ISP-10, SW1 RESET, U1 ATmega8-16PU, Y1 12MHz

Commit message: update: I have modified PCB design
Parts:
- Y1: footprint Crystal:Resonator-2Pin_W10.0mm_H5.0mm -> Crystal:Crystal_HC49-U_Vertical
Changed lines of the file:
@@
 F 0 "Y1" V 3554 2588 50  0000 L CNN
 F 1 "12MHz" V 3645 2588 50  0000 L CNN
-F 2 "Crystal:Resonator-2Pin_W10.0mm_H5.0mm" H 3600 2500 50  0001 C CNN
+F 2 "Crystal:Crystal_HC49-U_Vertical" H 3600 2500 50  0001 C CNN
 F 3 "~" H 3600 2500 50  0001 C CNN
 	1    3600 2500
@@
 Wire Wire Line
 	2300 2200 2600 2200
+$Comp
+L usbasp:LOGO #G1
+U 1 1 5DCA1D78
+P 2250 7050
+F 0 "#G1" H 2250 6620 60  0001 C CNN
+F 1 "LOGO" H 2250 7480 60  0001 C CNN
+F 2 "usbasp:logo_v2" H 2250 7050 50  0001 C CNN
+F 3 "" H 2250 7050 50  0001 C CNN
+	1    2250 7050
+	1    0    0    -1
+$EndComp
 $EndSCHEMATC
